File: kicad/rv8_cpu/rv8_cpu.kicad_sch (KiCad schematic)
At the start: 28 parts, among them J1 Conn_02x20_Odd_Even, U1 74LS161, U10 74LS574, U11 74LS161, U12 74LS161, U13 74LS283, U14 74LS283, U15 74HC86, U16 74LS157, U17 74LS157, U18 74HC138, U19 74HC245, U2 74LS161, U20 74HC74, U21 74HC74, U22 74LS08, U23 74LS32, U24 74HC138, U25 74LS157, U26 28C256, U27 KM62256CLP, U3 74LS161, U4 74LS161, U5 74LS574, U6 74LS574, U7 74LS574, U8 74LS574, U9 74LS574

Commit message: Fix KiCad schematic: verify all nets match circuit design
- 398 net connections, 180 unique nets
- 18/18 design verification checks pass
- PC carry chain, ALU carry, pointer carry correct
- Address decode, memory buses, control signals verified
- Added netlist.txt (human-readable net reference)
- U25 repurposed: clock mux + partial high-byte addr mux
- Note: A[15:8] driven by control logic (not chip-level mux)
Parts:
- removed U19: 74HC245, symbol 74xx:74HC245
- removed U20, U21: 74HC74, symbol 74xx:74HC74
- added U19: 74LS245, symbol 74xx:74LS245
- added U20, U21: 74LS74, symbol 74xx:74LS74
Other:
- note added: "ALU (U13-U14: 74HC283) + XOR (U15: 74HC86)"
- note added: "CONTROL: DECODE(U18) BUF(U19) FLAGS(U20-U21) AND(U22) OR(U23) ADDR_DEC(U24)"
- note added: "IR (U5-U6) + REGISTERS (U7=a0, U8=t0, U9=sp, U10=pg)"
- note added: "MEMORY: ROM(U26) RAM(U27) + EXPANSION CONNECTOR(J1)"
- note added: "POINTER (U11-U12) + ADDRESS MUX (U16-U17) + CLOCK MUX (U25)"
- note added: "PROGRAM COUNTER (U1-U4: 74HC161 ×4)"
- note removed: "ALU (U13-U15)"
- note removed: "CONTROL (U18-U23) + DECODE (U24)"
- note removed: "IR (U5-U6) + REGISTERS (U7-U10)"
- note removed: "MEMORY (U26-U27) + CONNECTOR (J1)"
- note removed: "POINTER (U11-U12) + ADDRESS MUX (U16-U17-U25)"
- note removed: "PROGRAM COUNTER (U1-U4)"

Commit message: Optimize KiCad: labels at pin endpoints, 364/364 connected
Other:
- note removed: "ALU (U13-U14: 74HC283) + XOR (U15: 74HC86)"
- note removed: "CONTROL: DECODE(U18) BUF(U19) FLAGS(U20-U21) AND(U22) OR(U23) ADDR_DEC(U24)"
- note removed: "IR (U5-U6) + REGISTERS (U7=a0, U8=t0, U9=sp, U10=pg)"
- note removed: "MEMORY: ROM(U26) RAM(U27) + EXPANSION CONNECTOR(J1)"
- note removed: "POINTER (U11-U12) + ADDRESS MUX (U16-U17) + CLOCK MUX (U25)"
- note removed: "PROGRAM COUNTER (U1-U4: 74HC161 ×4)"

Commit message: KiCad schematic v2: chip wiring diagram with wires + labels
- 28 symbols, 387 wires, 364 net labels
- Each pin has a wire stub + label showing connection
- Organized by function (6 rows)
- Exported: PDF + SVG for easy viewing
Other:
- note added: "ALU"
- note added: "CONTROL + ADDRESS DECODE"
- note added: "INSTRUCTION REGISTER + REGISTERS"
- note added: "POINTER + ADDRESS MUX + CLOCK"
- note added: "PROGRAM COUNTER"
- note added: "ROM + RAM + CONNECTOR"
- title: RV8 CPU Board -> RV8 CPU Board — Chip Wiring Diagram

Commit message: KiCad v3: human-centric data-flow layout, Verilog signal names
- Layout follows CPU pipeline: Fetch → Decode → Execute → Memory → Control
- Signal names match rv8_cpu.v (pc_inc, alu_result, ptr_out, etc.)
- 5 labeled sections with flow numbers ①②③④⑤
- Exported PDF + SVG for easy viewing
Other:
- note added: "① FETCH: Clock → PC → Address Mux → ROM/RAM"
- note added: "② DECODE: Data Bus → IR → Unit Decode / Address Decode"
- note added: "③ EXECUTE: a0 + operand → ALU → result → Registers"
- note added: "④ MEMORY: Pointer → Bus Buffer → External (40-pin)"
- note added: "⑤ CONTROL: Flags → Logic Gates → State Machine"
- note removed: "ALU"
- note removed: "CONTROL + ADDRESS DECODE"
- note removed: "INSTRUCTION REGISTER + REGISTERS"
- note removed: "POINTER + ADDRESS MUX + CLOCK"
- note removed: "PROGRAM COUNTER"
- note removed: "ROM + RAM + CONNECTOR"
- title: RV8 CPU Board — Chip Wiring Diagram -> RV8 CPU — Chip Wiring (Data Flow View)

Commit message: Add dataflow diagram + TTL schematic PDF, update KiCad project
Parts:
- U27: footprint (none) -> Package_DIP:DIP-28_W15.24mm
Connections:
- net A0: now also J1.37 (Pin_37), U26.20 (~{CS}), U27.1 (A14)
- net A1: now also J1.38 (Pin_38), U16.12 (Zd), U26.22 (~{OE}), U27.26 (A13)
- net A10: now also J1.27 (Pin_27), U26.25 (A8), U27.6 (A4)
- net A11: now also J1.28 (Pin_28), U26.3 (A7), U27.7 (A3)
- net A12: now also J1.25 (Pin_25), J1.32 (Pin_32), U17.7 (Zb), U26.23 (A11), U26.4 (A6), U27.3 (A7), U27.8 (A2)
- net A13: now also J1.26 (Pin_26), U26.5 (A5), U27.9 (A1)
- net A14: now also J1.23 (Pin_23), U24.6 (E2), U26.6 (A4), U27.10 (A0)
- net A15: now also J1.24 (Pin_24), U24.5 (~{E1})
- net A2: now also J1.35 (Pin_35), U16.9 (Zc), U26.27 (~{WE}), U27.2 (A12)
- net A3: now also J1.33 (Pin_33), J1.36 (Pin_36), U16.7 (Zb), U26.1 (A14), U27.21 (A10), U27.23 (A11)
- net A5: now also J1.30 (Pin_30), J1.31 (Pin_31), J1.34 (Pin_34), U17.12 (Zd), U17.9 (Zc), U26.2 (A12), U26.24 (A9), U26.26 (A13), U27.24 (A9), U27.25 (A8), U27.5 (A5)
- net A8: now also J1.29 (Pin_29), U26.21 (A10), U27.4 (A6)
- net CLK: now also J1.11 (Pin_11), U1.5 (D2), U11.5 (D2), U12.5 (D2), U2.5 (D2), U3.5 (D2), U4.5 (D2)
- net D0: now also J1.21 (Pin_21), U1.1 (~{MR}), U10.1 (OE), U11.1 (~{MR}), U12.1 (~{MR}), U5.1 (OE), U6.1 (OE), U8.1 (OE), U9.1 (OE)
- net D1: now also J1.22 (Pin_22), U10.11 (Cp), U5.11 (Cp), U6.11 (Cp), U8.11 (Cp), U9.11 (Cp)
- net D10: now also U3.2 (CP)
- net D11: now also U3.10 (CET)
- net D12: now also U4.1 (~{MR})
- net D14: now also U4.2 (CP)
- net D15: now also U4.10 (CET)
- net D2: now also J1.19 (Pin_19), U1.2 (CP), U11.2 (CP), U12.2 (CP), U27.27 (~{WE})
- net D3: now also J1.20 (Pin_20), U1.10 (CET), U10.9 (D7), U11.10 (CET), U12.10 (CET), U19.11 (B7), U27.22 (~{OE}), U5.9 (D7), U6.9 (D7), U8.9 (D7), U9.9 (D7)
- net D4: now also J1.17 (Pin_17), U10.8 (D6), U19.12 (B6), U2.1 (~{MR}), U5.8 (D6), U6.8 (D6), U8.8 (D6), U9.8 (D6)
- net D5: now also J1.18 (Pin_18), U10.7 (D5), U19.13 (B5), U27.20 (~{CS}), U5.7 (D5), U6.7 (D5), U8.7 (D5), U9.7 (D5)
- net D6: now also J1.15 (Pin_15), U10.6 (D4), U19.14 (B4), U2.2 (CP), U5.6 (D4), U6.6 (D4), U8.6 (D4), U9.6 (D4)
- net D7: now also J1.16 (Pin_16), U10.5 (D3), U19.15 (B3), U2.10 (CET), U27.19 (Q7), U5.5 (D3), U6.5 (D3), U8.5 (D3), U9.5 (D3)
- net D8: now also U3.1 (~{MR})
- net HALT: now also J1.7 (Pin_7)
- net IRQ_N: now also J1.10 (Pin_10)
- net NMI_N: now also J1.9 (Pin_9)
- net OSC_3M5: now also U25.1 (S)
- net PC0: now also U16.1 (S)
- net PC1: now also U16.14 (I0d)
- net PC2: now also U16.11 (I0c)
- net PC3: now also U16.5 (I0b)
- net PC4: now also U17.1 (S)
- net PC5: now also U17.14 (I0d)
- net PC6: now also U17.11 (I0c)
- net PC7: now also U17.5 (I0b)
- net RST_N: now also J1.12 (Pin_12), U1.3 (D0), U11.3 (D0), U12.3 (D0), U2.3 (D0), U3.3 (D0), U4.3 (D0)
- net RUN_N: now also U25.2 (I0a)
- net SYNC: now also J1.8 (Pin_8)
- net U1_TC: now also U1.15 (TC), U2.6 (D3)
- net U2_TC: now also U2.15 (TC), U3.6 (D3)
- net U3_TC: now also U3.15 (TC), U4.6 (D3)
- net a0_clk: now also U7.3 (D1)
- net a0_out0: now also U13.2 (B2)
- net a0_out1: now also U13.6 (B1)
- net a0_out3: now also U13.12 (A4), U7.12 (Q7)
- net a0_out4: now also U14.2 (B2), U7.13 (Q6)
- net a0_out5: now also U14.6 (B1), U7.14 (Q5)
- net a0_out6: now also U7.15 (Q4)
- net a0_out7: now also U14.12 (A4), U7.16 (Q3)
- net addr_sel: now also U16.2 (I0a), U17.2 (I0a)
- net alu_b0: now also U13.3 (A2)
- net alu_b1: now also U13.5 (A1)
- net alu_b3: now also U13.7 (C0)
- net alu_b4: now also U14.3 (A2)
- net alu_b5: now also U14.5 (A1)
- net alu_b7: now also U14.7 (C0)
- net alu_result0: now also U7.1 (OE)
- net alu_result1: now also U7.11 (Cp)
- net alu_result3: now also U7.9 (D7)
- net alu_result4: now also U7.8 (D6)
- net alu_result5: now also U7.7 (D5)
- net alu_result6: now also U7.6 (D4)
- net alu_result7: now also U7.5 (D3)
- net branch_en_n: now also U18.10 (~{Y5})
- net buf_dir: now also U19.3 (A1)
- net buf_en_n: now also U19.2 (A0)
- net carry_in: now also U13.11 (B4)
- net carry_mid: now also U13.9 (C4), U14.11 (B4)
- net carry_out: now also U14.9 (C4)
- net data_int0: now also U19.19 (CE)
- net data_int1: now also U19.1 (A->B)
- net data_int3: now also U19.9 (A7)
- net data_int4: now also U19.8 (A6)
- net data_int5: now also U19.7 (A5)
- net data_int6: now also U19.6 (A4)
- net data_int7: now also U19.5 (A3)
- net exec_n: now also U18.3 (A2)
- net imm_en_n: now also U18.7 (~{Y7})
- net io_cs_n: now also U24.11 (~{Y4})
- net ir_load0: now also U5.3 (D1)
- net ir_load1: now also U6.3 (D1)
- net ldst_en_n: now also U18.9 (~{Y6})
- net mem_rd_n: now also J1.13 (Pin_13), U26.9 (A1), U27.15 (Q3)
- net mem_wr_n: now also J1.14 (Pin_14), U27.13 (Q2)
- net opcode3: now also U5.12 (Q7)
- net opcode4: now also U5.13 (Q6)
- net opcode5: now also U5.14 (Q5)
- net opcode6: now also U18.6 (E2), U5.15 (Q4)
- net opcode7: now also U18.5 (~{E1}), U5.16 (Q3)
- net operand3: now also U6.12 (Q7)
- net operand4: now also U6.13 (Q6)
- net operand5: now also U6.14 (Q5)
- net operand6: now also U6.15 (Q4)
- net operand7: now also U6.16 (Q3)
- net pc_inc: now also U1.6 (D3)
- net pc_load_n: now also U1.9 (~{PE}), U2.9 (~{PE}), U3.9 (~{PE}), U4.9 (~{PE})
- net pg_clk: now also U10.3 (D1)
- net pg_out3: now also U10.12 (Q7)
- net pg_out4: now also U10.13 (Q6)
- net pg_out5: now also U10.14 (Q5)
- net pg_out6: now also U10.15 (Q4)
- net pg_out7: now also U10.16 (Q3)
- net ph_load_n: now also U12.9 (~{PE})
- net pl_load_n: now also U11.9 (~{PE})
- net ptr_en_n: now also U18.12 (~{Y3})
- net ptr_inc: now also U11.6 (D3)
- net ptr_tc: now also U11.15 (TC), U12.6 (D3)
- net ram_ce_n: now also U27.17 (Q5)
- net ram_cs1_n: now also U24.7 (~{Y7})
- net rom_ce_n: now also U26.10 (A0)
- net rom_cs6_n: now also U24.13 (~{Y2})
- net rom_cs7_n: now also U24.14 (~{Y1})
- net shift_en_n: now also U18.11 (~{Y4})
- net slot0_n: now also U24.9 (~{Y6})
- net slot1_n: now also U24.10 (~{Y5})
- net sp_clk: now also U9.3 (D1)
- net sp_out3: now also U9.12 (Q7)
- net sp_out4: now also U9.13 (Q6)
- net sp_out5: now also U9.14 (Q5)
- net sp_out6: now also U9.15 (Q4)
- net sp_out7: now also U9.16 (Q3)
- net sys_en_n: now also U18.14 (~{Y1})
- net t0_clk: now also U8.3 (D1)
- net t0_out3: now also U8.12 (Q7)
- net t0_out4: now also U8.13 (Q6)
- net t0_out5: now also U8.14 (Q5)
- net t0_out6: now also U8.15 (Q4)
- net t0_out7: now also U8.16 (Q3)
- new net +5V: U18.2 (A1), U24.2 (A1), U26.8 (A2)
- new net GND: U10.2 (D0), U24.3 (A2), U25.11 (I0c), U25.14 (I0d), U25.5 (I0b), U5.2 (D0), U6.2 (D0), U7.2 (D0), U8.2 (D0), U9.2 (D0)
